File: camera_control_pcb/board.brd (EAGLE design)
At the start: 160 x 100 mm, 20 parts, among them Q1 MPSA42

Commit message: Fix switch sizes to 10mm
Parts:
- removed S11: (no value), switch-omron:B3F-40XX
- S10, S2, S3, S4, S5, S6, S7, S8, S9: device switch-omron:B3F-40XX -> switch-omron:B3F-10XX
- moved S3 286.8 mm to (-87.6, 62.2)
- moved S7 261.4 mm to (-48.3, 62.2)
- moved S8 235.9 mm to (-58.4, 62.2), turned to 0 degrees
- moved S9 214.1 mm to (-68.6, 62.2)
- moved S2 203.4 mm to (-77.5, 62.2)
- moved S4 179.9 mm to (-17.8, 62.2)
- moved S10 178.6 mm to (-17.8, 71.1)
- moved S5 176.8 mm to (-27.9, 62.2)
- moved S1 163.5 mm to (-67.3, 7.62)
- moved TM3 163.2 mm to (-50.8, 38.1)
- moved S6 162.4 mm to (-38.1, 62.2)
- moved TM2 131.8 mm to (-50.8, 25.4)
- moved ARDUINO_NANO1 119.6 mm to (-33.0, 10.2), turned to 0 degrees
- moved H1 100.7 mm to (-19.1, 52.1)
- moved H3 87.6 mm to (-44.5, 52.1)
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Connections:
- new net N$20: S2.2, S3.1
- new net N$21: S3.2, S4.1
- new net N$22: S4.2, S5.1
- new net N$23: S6.1
- new net N$24: S6.2, S7.1, S8.1
- new net N$25: S8.2, S9.1
- new net N$26: S10.1, S9.2
- net N$10: now also S8.3; no longer S9.3
- net N$11: now also S9.3; no longer S10.3
- net N$12: now also S10.3; no longer S11.3
- net N$13: now also S2.4; no longer S2.3
- net N$14: no longer S4.3
- net N$3: no longer S10.1, S11.1, S11.2, S2.1, S2.2, S3.1, S3.2, S4.1, S4.2, S5.1, S6.1, S6.2, S7.1, S7.2, S8.1, S9.1, S9.2
- net N$6: now also S6.3; no longer S7.3
- net N$7: now also S4.3; no longer S5.3
- net N$8: now also S5.3; no longer S6.3
- net N$9: now also S7.3; no longer S8.3

Commit message: Example Board Layout with 11 vias
Parts:
- added LED1: (no value), led:LED5MM
- added S11: (no value), switch-omron:B3F-10XX
- moved TM2 203.0 mm to (149.9, 55.9), turned to 90 degrees
- moved R1 192.4 mm to (144.8, 6.35), turned to 180 degrees
- moved TM3 187.5 mm to (135.9, 55.9), turned to 270 degrees
- moved Q1 173.3 mm to (129.5, 6.35), turned to 180 degrees
- moved S3 165.4 mm to (77.5, 52.1), turned to 180 degrees
- moved S6 158.0 mm to (119.4, 74.9), turned to 180 degrees
- moved S7 148.5 mm to (97.8, 88.9), turned to 180 degrees
- moved S9 148.0 mm to (76.2, 92.7), turned to 180 degrees
- moved H3 140.8 mm to (92.7, 20.3), turned to 180 degrees
- moved R4 140.3 mm to (83.8, 7.62), turned to 180 degrees
- moved S4 138.6 mm to (120.7, 54.6), turned to 180 degrees
- moved S2 126.9 mm to (45.7, 31.8), turned to 180 degrees
- moved S10 115.0 mm to (96.5, 58.4), turned to 180 degrees
- moved S1 115.0 mm to (15.2, 87.6), turned to 180 degrees
- moved S8 110.0 mm to (48.3, 88.9), turned to 180 degrees
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Connections:
- new net N$27: S11.2, S4.1
- new net N$28: ARDUINO_NANO1.1, LED1.A
- net N$14: now also S11.3
- net N$21: now also S11.1; no longer S4.1
- net N$3: now also LED1.K
Routing:
- net N$3: track 0.00 -> 404.9 mm, vias 0 -> 3
- net N$18: track 0.00 -> 193.1 mm
- net N$17: track 0.00 -> 170.7 mm, vias 0 -> 2
- net N$19: track 0.00 -> 161.5 mm
- net N$14: track 0.00 -> 148.5 mm
- net N$6: track 0.00 -> 129.3 mm, vias 0 -> 2
- net N$9: track 0.00 -> 111.5 mm
- net N$2: track 0.00 -> 111.0 mm
- net N$7: track 0.00 -> 107.3 mm, vias 0 -> 2
- net N$12: track 0.00 -> 92.9 mm
- net N$16: track 0.00 -> 78.6 mm
- net N$15: track 0.00 -> 75.8 mm
- net N$11: track 0.00 -> 74.7 mm, vias 0 -> 1
- net N$24: track 0.00 -> 74.5 mm
- net N$22: track 0.00 -> 71.2 mm
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
Commit message: No vias board layout
Parts:
- moved TM3 122.1 mm to (14.0, 49.5)
- moved TM2 118.3 mm to (31.8, 49.5)
- moved S1 81.9 mm to (55.9, 16.5)
- moved R1 62.2 mm to (82.5, 7.62), turned to 0 degrees
- moved ARDUINO_NANO1 49.0 mm to (59.7, 63.5)
- moved S8 43.3 mm to (91.4, 91.4)
- moved S9 39.5 mm to (115.6, 95.2)
- moved S2 37.6 mm to (82.5, 39.4)
- moved S7 37.0 mm to (134.6, 92.7)
- moved S5 33.4 mm to (81.3, 69.8)
- moved LED1 29.6 mm to (29.2, 94.0)
- moved S11 26.9 mm to (132.1, 39.4)
- moved S6 26.9 mm to (146.1, 78.7)
- moved S10 26.9 mm to (123.2, 62.2)
- moved S3 26.9 mm to (104.1, 55.9)
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Routing:
- net N$18: track 193.1 -> 69.6 mm
- net N$3: track 404.9 -> 281.4 mm, vias 3 -> 0
- net N$19: track 161.5 -> 46.2 mm
- net N$2: track 111.0 -> 38.7 mm
- net N$14: track 148.5 -> 77.9 mm
- net N$17: track 170.7 -> 120.7 mm, vias 2 -> 0
- net N$15: track 75.8 -> 42.3 mm
- net N$9: track 111.5 -> 80.3 mm
- net N$6: track 129.3 -> 101.8 mm, vias 2 -> 0
- net N$5: track 63.1 -> 42.1 mm
- net N$8: track 36.4 -> 18.7 mm
- net N$10: track 55.4 -> 37.9 mm
- net N$11: track 74.7 -> 59.3 mm, vias 1 -> 0
- net N$4: track 48.4 -> 63.3 mm
- net N$16: track 78.6 -> 92.2 mm
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