File: pcb/board.brd (EAGLE design)
At the start: 160 x 100 mm, 21 parts, among them Q1 MPSA42

Commit message: Clean-up repository
Parts:
- removed H1, H2, H3: MOUNT-PAD-ROUND4.1, holes:4,1-PAD
- removed R4: (no value), rcl:0204V
- removed TM2: (no value), Bourns PTA series:SLIDEPOT-75
- added CAM/PIN1, CAM/PIN2, CAM/PIN6, GND, POT1, POT2, POT3, PWR: (no value), wirepad:1,6/0,8
- added CON1: (no value), db25:D-25F
- added R2: (no value), rcl:0204V
- added U$1, U$2, U$3, U$4: (no value), holes:2,8
- added X1, X2: DIN8, con-din8:DIN8
- S1: value (none) -> 471002268142_PANELTHICKNESS1.5MM; device switch-omron:B3F-40XX -> power_switch:47100226814X_PANELTHICKNESS1.5MM
- moved S1 131.0 mm to (80.2, -22.6), turned to 0 degrees
- moved S3 98.4 mm to (109.2, 17.8)
- moved TM3 96.7 mm to (27.9, 45.7)
- moved S11 96.4 mm to (109.2, 83.8)
- moved S9 89.5 mm to (109.2, 67.3)
- moved LED1 89.2 mm to (20.3, 92.7)
- moved Q1 85.3 mm to (67.4, 42.2), turned to 90 degrees
- moved S5 78.5 mm to (109.2, 34.3)
- moved S10 77.2 mm to (92.7, 83.8)
- moved S2 76.5 mm to (92.7, 17.8)
- moved R1 76.1 mm to (66.0, 62.8)
- moved S8 69.5 mm to (92.7, 67.3)
- moved S4 67.0 mm to (92.7, 34.3)
- moved S7 62.6 mm to (109.2, 50.8)
- moved S6 46.0 mm to (92.7, 50.8)
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Connections:
- new net N$20: X1.P$2
- new net N$21: X1.P$1
- new net N$22: CON1.2, X2.P$2
- new net N$23: CON1.6, X2.P$7
- new net N$24: CON1.1, X2.P$1
- new net N$25: S1.1
- net GND: now also CAM/PIN1.1, GND.1, POT3.1, S1.2; no longer H3.B4,1, TM2.B
- net N$1: now also X1.P$7; no longer S1.3
- net N$13: now also CAM/PIN6.1, PWR.1; no longer H1.B4,1, S1.1
- net N$14: now also R1.1; no longer R4.1
- net N$15: now also R1.2; no longer R4.2
- net N$16: now also ARDUINO_NANO1.5; no longer ARDUINO_NANO1.6
- net N$17: now also ARDUINO_NANO1.6, POT2.1; no longer ARDUINO_NANO1.5, TM2.WIPER
- net N$18: now also CAM/PIN2.1, R2.1; no longer H2.B4,1, R1.1
- net N$2: now also POT1.1, R2.2; no longer R1.2, TM2.A
Routing:
- net GND: track 309.0 -> 0.45 mm, vias 1 -> 0
- net N$2: track 94.4 -> 308.1 mm
- net N$18: track 224.0 -> 54.5 mm
- net N$13: track 154.6 -> 26.7 mm
- net N$14: track 100.0 -> 35.5 mm
- net N$17: track 61.8 -> 6.49 mm
- net N$15: track 71.5 -> 19.4 mm
- net N$12: track 21.0 -> 66.9 mm
- net N$19: track 24.8 -> 62.4 mm
- net N$11: track 17.4 -> 48.5 mm
- net N$10: track 32.9 -> 58.5 mm
- net N$8: track 20.6 -> 43.0 mm
- net N$16: track 77.4 -> 55.3 mm
- net N$9: track 29.9 -> 40.7 mm
- net N$5: track 42.3 -> 32.7 mm
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- added copper zone on layer 16, net GND
Other:
- board size 160 x 100 mm -> 127 x 101.6 mm
