File: pcb.reduced/board.brd (EAGLE design)
At the start: 127 x 101.6 mm, 28 parts, among them Q1 MPSA42

Commit message: update gerber files
Parts:
- flipped TM3 to the bottom
Routing:
- net N$16: track 54.5 -> 50.9 mm
